Commit message: the simulation can control the joint of robot but it wrong position, not like in the hardware
Signed-off-by: VuongAdonis <vuong03062003@gmail.com>

File: ros2_ws/install/simulation/share/simulation/urdf/robot.urdf (robot description, URDF)
Before this commit: robot Dog robot, 17 links, 16 joints
Joints:
- removed joint thigh_joint_fl_to_shoulder_rl
- added joint thigh_joint_rl_to_shoulder_rl: type revolute, parent shoulder_link_rl, child thigh_link_rl, origin xyz=0 ${-shoul_len} 0, axis 0 1 0, limit lower=${-limit_thigh} upper=${limit_thigh} effort=1000.0 velocity=0.5

Commit message: add code to check if 1 encoder_pos is oke, don't need to send again
Signed-off-by: VuongAdonis <vuong03062003@gmail.com>

File: ros2_ws/install/simulation/share/simulation/urdf/robot.urdf (robot description, URDF)
Before this commit: robot Dog robot, 17 links, 16 joints
Links:
- link shoulder_link_fr: mass 1e-5 -> ${mass}
Joints:
- joint shoulder_joint_fl_to_base: origin xyz=${0.5*body_len + link_radius} -0.75 0 -> xyz=${0.5*body_len + link_radius} -0.75 ${high_of_Robot}
- joint shoulder_joint_fr_to_base: origin xyz=${0.5*body_len + link_radius} 0.75 0 -> xyz=${0.5*body_len + link_radius} 0.75 ${high_of_Robot}
- joint shoulder_joint_rl_to_base: origin xyz=${-0.5*body_len + link_radius} -0.75 0 -> xyz=${-0.5*body_len + link_radius} -0.75 ${high_of_Robot}
- joint shoulder_joint_rr_to_base: origin xyz=${-0.5*body_len + link_radius} 0.75 0 -> xyz=${-0.5*body_len + link_radius} 0.75 ${high_of_Robot}
